File: GeT_Computer.kicad_pcb (KiCad board)
At the start: 4 copper layers, 85 x 56 mm, 113 parts, among them J1 USB_C_Receptacle_USB2.0_16P, J2 DE15_Socket_HighDensity_Mount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, J3 Micro_SD_Card, J4 Mini-DIN-6, J5 Conn_02x03_Counter_Clockwise, J6 Conn_02x12_Odd_Even, P1 RB1-125BAG1A, U1 NCP1117-3.3_SOT223, U2 RPI_RMC20452T, U3 APS6404L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

Commit message: Add final version of the project that was printed and assembled
Parts:
- added REF**: MountingHole_2.7mm_M2.5, GeT_Footprints_Library:MountingHole_2.7mm_M2.5, F.Cu at (155.0, 61.0)
- added REF**: MountingHole_2.7mm_M2.5, GeT_Footprints_Library:MountingHole_2.7mm_M2.5, F.Cu at (97.0, 110.0)
- added REF**: MountingHole_2.7mm_M2.5, GeT_Footprints_Library:MountingHole_2.7mm_M2.5, F.Cu at (155.0, 110.0)
- added REF**: MountingHole_2.7mm_M2.5, GeT_Footprints_Library:MountingHole_2.7mm_M2.5, F.Cu at (97.0, 61.0)
- added TP1: TestPoint, TestPoint:TestPoint_Pad_D2.0mm, B.Cu at (131.0, 88.3)
- added TP2: TestPoint, TestPoint:TestPoint_Pad_D2.0mm, B.Cu at (128.0, 83.3)
- added TP3: TestPoint, TestPoint:TestPoint_Pad_D2.0mm, B.Cu at (131.1, 78.9)
Routing:
- net +1V1: track 30.9 -> 35.5 mm
