File: GeT_Computer.kicad_sch (KiCad schematic)
At the start: 113 parts, among them J1 USB_C_Receptacle_USB2.0_16P, J2 DE15_Socket_HighDensity_Mount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, J3 Micro_SD_Card, J4 Mini-DIN-6, J5 Conn_02x03_Counter_Clockwise, J6 Conn_02x12_Odd_Even, P1 RB1-125BAG1A, U1 NCP1117-3.3_SOT223, U2 RPI_RMC20452T, U3 APS6404L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

Commit message: Add final version of the project that was printed and assembled
Parts:
- added TP1, TP2, TP3: TestPoint, TestPoint:TestPoint_Pad_D2.0mm, symbol Connector:TestPoint
Connections:
- net +1V1: now also TP1.1, TP2.1, TP3.1
